File: OpenAmigaVideoHybrid.kicad_pcb (KiCad board)
At the start: 2 copper layers, 56.4 x 21.2 mm, 59 parts, among them J1 CONN_MAINBOARD, J2 SVIDEO_OUT, Q1 2N3904, Q2 2N3904, Q3 2N3904, Q4 2N3904, U1 AD724, Y2 4.433619M

Commit message: Some more stitching and we're done
Parts:
- moved J2 0.32 mm to (171.3, 107.3)
Routing:
- net GND: vias 3 -> 32
Changed lines of the file:
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@@
   (general
     (thickness 1.6)
-    (drawings 18)
-    (tracks 299)
+    (drawings 21)
+    (tracks 326)
     (zones 0)
     (modules 59)
@@
     (tags "capacitor handsolder")
     (attr smd)
-    (fp_text reference C11 (at 3.479 0) (layer B.SilkS)
+    (fp_text reference C11 (at 3.225 0) (layer B.SilkS)
       (effects (font (size 1 1) (thickness 0.15)) (justify mirror))
     )
@@
     (tags "capacitor handsolder")
     (attr smd)
-    (fp_text reference C18 (at 3.556 0) (layer B.SilkS)
+    (fp_text reference C18 (at 3.3655 0) (layer B.SilkS)
       (effects (font (size 1 1) (thickness 0.15)) (justify mirror))
     )
@@
     (tags "resistor handsolder")
     (attr smd)
-    (fp_text reference R31 (at 3.2385 -1.375833) (layer B.SilkS)
+    (fp_text reference R31 (at 3.6195 -2.074333) (layer B.SilkS)
       (effects (font (size 1 1) (thickness 0.15)) (justify mirror))
     )
@@
   )
   (module OpenAmigaVideoHybrid:Pin_Header_Straight_1x03-ModSilkS (layer B.Cu)
-    (at 171.577 107.3085 180)
+    (at 171.2595 107.315 180)
     (descr "Through hole straight pin header, 1x03, 2.54mm pitch, single row")
     (tags "Through hole pin header THT 1x03 2.54mm single row")
@@
     )
   )
-  (gr_text G (at 169.672 112.395) (layer B.SilkS)
+  (gr_line (start 138.938 109.1565) (end 139.446 109.1565) (layer B.SilkS) (width 0.15))
+  (gr_line (start 138.938 108.6485) (end 138.938 109.1565) (layer B.SilkS) (width 0.15))
+  (gr_line (start 139.5095 108.585) (end 138.938 109.1565) (layer B.SilkS) (width 0.15))
+  (gr_text G (at 173.4185 112.395) (layer B.SilkS)
     (effects (font (size 1 1) (thickness 0.15)) (justify mirror))
   )
-  (gr_text L (at 169.767238 109.855) (layer B.SilkS)
+  (gr_text L (at 173.513738 109.855) (layer B.SilkS)
     (effects (font (size 1 1) (thickness 0.15)) (justify mirror))
   )
-  (gr_text C (at 169.672 107.315) (layer B.SilkS)
+  (gr_text C (at 173.4185 107.315) (layer B.SilkS)
     (effects (font (size 1 1) (thickness 0.15)) (justify mirror))
   )
@@
     (effects (font (size 1 1) (thickness 0.15)) (justify mirror))
   )
-  (gr_text PAL (at 137.931 115.824) (layer B.SilkS)
+  (gr_text PAL (at 138.2395 115.951) (layer B.SilkS)
     (effects (font (size 1 1) (thickness 0.15)) (justify mirror))
   )
@@
   (via (at 145.923 113.6585) (size 0.8) (drill 0.6) (layers F.Cu B.Cu) (net 1))
   (via (at 145.923 109.8485) (size 0.8) (drill 0.6) (layers F.Cu B.Cu) (net 1))
+  (via (at 148.7805 111.7535) (size 0.8) (drill 0.6) (layers F.Cu B.Cu) (net 1))
+  (via (at 148.336 109.8485) (size 0.8) (drill 0.6) (layers F.Cu B.Cu) (net 1))
+  (via (at 148.7805 113.6585) (size 0.8) (drill 0.6) (layers F.Cu B.Cu) (net 1))
+  (via (at 143.51 116.078) (size 0.8) (drill 0.6) (layers F.Cu B.Cu) (net 1))
+  (via (at 145.923 116.078) (size 0.8) (drill 0.6) (layers F.Cu B.Cu) (net 1))
+  (via (at 148.59 118.364) (size 0.8) (drill 0.6) (layers F.Cu B.Cu) (net 1))
+  (via (at 148.59 121.031) (size 0.8) (drill 0.6) (layers F.Cu B.Cu) (net 1))
+  (via (at 145.923 118.3005) (size 0.8) (drill 0.6) (layers F.Cu B.Cu) (net 1))
+  (via (at 143.51 118.3005) (size 0.8) (drill 0.6) (layers F.Cu B.Cu) (net 1))
+  (via (at 143.51 121.031) (size 0.8) (drill 0.6) (layers F.Cu B.Cu) (net 1))
+  (via (at 135.89 118.364) (size 0.8) (drill 0.6) (layers F.Cu B.Cu) (net 1))
+  (via (at 130.81 118.364) (size 0.8) (drill 0.6) (layers F.Cu B.Cu) (net 1))
+  (via (at 137.16 115.3795) (size 0.8) (drill 0.6) (layers F.Cu B.Cu) (net 1))
+  (via (at 133.1595 113.157) (size 0.8) (drill 0.6) (layers F.Cu B.Cu) (net 1))
+  (via (at 139.5095 108.9025) (size 0.8) (drill 0.6) (layers F.Cu B.Cu) (net 1))
+  (via (at 137.2235 111.0615) (size 0.8) (drill 0.6) (layers F.Cu B.Cu) (net 1))
+  (via (at 132.6515 108.839) (size 0.8) (drill 0.6) (layers F.Cu B.Cu) (net 1))
+  (via (at 133.223 111.3155) (size 0.8) (drill 0.6) (layers F.Cu B.Cu) (net 1))
+  (via (at 128.905 108.839) (size 0.8) (drill 0.6) (layers F.Cu B.Cu) (net 1))
+  (via (at 122.9995 108.839) (size 0.8) (drill 0.6) (layers F.Cu B.Cu) (net 1))
+  (via (at 128.0795 111.506) (size 0.8) (drill 0.6) (layers F.Cu B.Cu) (net 1))
+  (via (at 128.0795 113.792) (size 0.8) (drill 0.6) (layers F.Cu B.Cu) (net 1))
+  (via (at 128.0795 116.0145) (size 0.8) (drill 0.6) (layers F.Cu B.Cu) (net 1))
+  (via (at 124.714 116.0145) (size 0.8) (drill 0.6) (layers F.Cu B.Cu) (net 1))
+  (via (at 123.444 111.506) (size 0.8) (drill 0.6) (layers F.Cu B.Cu) (net 1))
+  (via (at 120.396 111.506) (size 0.8) (drill 0.6) (layers F.Cu B.Cu) (net 1))
+  (via (at 120.396 117.2845) (size 0.8) (drill 0.6) (layers F.Cu B.Cu) (net 1))
+  (via (at 125.73 118.364) (size 0.8) (drill 0.6) (layers F.Cu B.Cu) (net 1))
+  (via (at 123.19 118.364) (size 0.8) (drill 0.6) (layers F.Cu B.Cu) (net 1))
   (segment (start 121.92 121.92) (end 124.46 124.46) (width 0.25) (layer F.Cu) (net 2) (status 20))
   (segment (start 121.92 119.389) (end 121.92 121.92) (width 0.25) (layer F.Cu) (net 2) (status 10))
@@
   (segment (start 131.613 107.8865) (end 131.613 109.960833) (width 0.25) (layer B.Cu) (net 6) (status 30))
   (segment (start 131.613 109.960833) (end 131.593167 109.960833) (width 0.25) (layer B.Cu) (net 6) (status 30))
-  (segment (start 131.613 109.960833) (end 131.613 110.068) (width 0.25) (layer B.Cu) (net 6) (status 30))
-  (segment (start 131.613 110.068) (end 129.032 112.649) (width 0.25) (layer B.Cu) (net 6) (status 10))
-  (segment (start 129.032 112.649) (end 129.032 115.443) (width 0.25) (layer B.Cu) (net 6))
-  (segment (start 129.032 115.443) (end 129.032 115.189) (width 0.25) (layer B.Cu) (net 6))
-  (segment (start 129.032 122.174) (end 129.032 115.443) (width 0.25) (layer B.Cu) (net 6))
-  (segment (start 130.048 123.19) (end 129.032 122.174) (width 0.25) (layer B.Cu) (net 6))
-  (segment (start 134.62 124.46) (end 133.35 123.19) (width 0.25) (layer B.Cu) (net 6) (status 10))
+  (segment (start 131.613 110.068) (end 131.613 109.960833) (width 0.25) (layer B.Cu) (net 6))
   (segment (start 133.35 123.19) (end 130.048 123.19) (width 0.25) (layer B.Cu) (net 6))
+  (segment (start 134.62 124.46) (end 133.35 123.19) (width 0.25) (layer B.Cu) (net 6))
+  (segment (start 130.048 123.19) (end 128.905 122.047) (width 0.25) (layer B.Cu) (net 6))
+  (segment (start 128.905 122.047) (end 128.905 112.776) (width 0.25) (layer B.Cu) (net 6))
+  (segment (start 128.905 112.776) (end 131.613 110.068) (width 0.25) (layer B.Cu) (net 6))
   (segment (start 136.1985 109.960833) (end 136.1985 107.8865) (width 0.25) (layer B.Cu) (net 11) (status 30))
+  (segment (start 136.1985 110.0545) (end 134.112 112.141) (width 0.25) (layer B.Cu) (net 11))
+  (segment (start 136.1985 109.960833) (end 136.1985 110.0545) (width 0.25) (layer B.Cu) (net 11))
+  (segment (start 134.112 112.141) (end 131.064 112.141) (width 0.25) (layer B.Cu) (net 11))
+  (segment (start 145.542 122.682) (end 147.32 124.46) (width 0.25) (layer B.Cu) (net 11))
   (segment (start 130.302 122.682) (end 145.542 122.682) (width 0.25) (layer B.Cu) (net 11))
-  (segment (start 129.54 121.92) (end 130.302 122.682) (width 0.25) (layer B.Cu) (net 11))
-  (segment (start 136.1985 109.960833) (end 136.1985 110.0545) (width 0.25) (layer B.Cu) (net 11) (status 30))
-  (segment (start 134.112 112.141) (end 131.064 112.141) (width 0.25) (layer B.Cu) (net 11))
-  (segment (start 145.542 122.682) (end 147.32 124.46) (width 0.25) (layer B.Cu) (net 11) (status 20))
-  (segment (start 136.1985 110.0545) (end 134.112 112.141) (width 0.25) (layer B.Cu) (net 11) (status 10))
-  (segment (start 131.064 112.141) (end 129.54 113.665) (width 0.25) (layer B.Cu) (net 11))
-  (segment (start 129.54 113.665) (end 129.54 121.92) (width 0.25) (layer B.Cu) (net 11))
+  (segment (start 131.064 112.141) (end 129.413 113.792) (width 0.25) (layer B.Cu) (net 11))
+  (segment (start 129.413 121.793) (end 130.302 122.682) (width 0.25) (layer B.Cu) (net 11))
+  (segment (start 129.413 113.792) (end 129.413 121.793) (width 0.25) (layer B.Cu) (net 11))
   (segment (start 147.32 121.92) (end 149.86 124.46) (width 0.25) (layer F.Cu) (net 12) (status 20))
   (segment (start 147.32 119.389) (end 147.32 121.92) (width 0.25) (layer F.Cu) (net 12) (status 10))
@@
   (segment (start 157.48 119.389) (end 157.48 121.92) (width 0.25) (layer F.Cu) (net 16) (status 10))
   (segment (start 136.1985 114.1095) (end 136.1985 112.035166) (width 0.25) (layer B.Cu) (net 16) (status 30))
-  (segment (start 157.734 122.174) (end 160.02 124.46) (width 0.25) (layer B.Cu) (net 16) (status 20))
-  (segment (start 130.6195 114.1095) (end 130.048 114.681) (width 0.25) (layer B.Cu) (net 16))
-  (segment (start 130.048 114.681) (end 130.048 121.7295) (width 0.25) (layer B.Cu) (net 16))
-  (segment (start 136.1985 114.1095) (end 130.6195 114.1095) (width 0.25) (layer B.Cu) (net 16) (status 10))
-  (segment (start 130.048 121.7295) (end 130.4925 122.174) (width 0.25) (layer B.Cu) (net 16))
+  (segment (start 130.6195 114.1095) (end 129.921 114.808) (width 0.25) (layer B.Cu) (net 16))
+  (segment (start 157.734 122.174) (end 160.02 124.46) (width 0.25) (layer B.Cu) (net 16))
+  (segment (start 136.1985 114.1095) (end 130.6195 114.1095) (width 0.25) (layer B.Cu) (net 16))
+  (segment (start 129.921 121.6025) (end 130.4925 122.174) (width 0.25) (layer B.Cu) (net 16))
+  (segment (start 129.921 114.808) (end 129.921 121.6025) (width 0.25) (layer B.Cu) (net 16))
   (segment (start 130.4925 122.174) (end 157.734 122.174) (width 0.25) (layer B.Cu) (net 16))
   (segment (start 160.02 121.92) (end 162.56 124.46) (width 0.25) (layer F.Cu) (net 17) (status 20))
